File: hardware/1280_modem.kicad_pcb (KiCad board)
At the start: 4 copper layers, 38 x 53 mm, 95 parts, among them IC1 SX1281IMLTRT, IC2 SKY65383-11, IC3 LMR50410Y3, J1 jst_sh 6, J2 Conn_Coaxial, J3 USB_C_Receptacle_USB2.0, J4 jst gh 4, J5 jst gh 6, Q1 AO3401A, Q2 AO3401A, U1 STM32U575CGTx, U2 TPS7A20285PDBVR, U3 USBLC6-2SC6, U4 TCAN334, Y1 48MHz, Y2 52MHz

Commit message: final (?) bom
Parts:
- C15, C16, C17: value 10p -> 18p
- C21, C22: value 13p -> 18p
- C25, C29: value 4u7 -> 100n
- C27: value 10u -> 1u
- C3, C5: value 14p -> 18p
- C6: value 100n -> 10n
- C7: value 470n -> 1u
- Q1, Q2: value AO3401A -> DMP3056L-7
- U4: value TCAN334 -> TCAN334GDCN
Changed lines of the file:
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@@
 			)
 		)
-		(property ki_fp_filters "MountingHole*Pad*")
-		(sheetname "Root")
-		(sheetfile "1280_modem.kicad_sch")
 		(attr exclude_from_pos_files)
 		(fp_circle
@@
 			(pinfunction "1")
 			(pintype "input")
+			(zone_connect 2)
 		)
 		(pad "1" thru_hole circle
@@
 			(pinfunction "1")
 			(pintype "input")
+			(zone_connect 2)
 		)
 		(pad "1" thru_hole circle
@@
 			(pinfunction "1")
 			(pintype "input")
+			(zone_connect 2)
 		)
 		(pad "1" thru_hole circle
@@
 			(pinfunction "1")
 			(pintype "input")
+			(zone_connect 2)
 		)
 		(pad "1" thru_hole circle
@@
 			(pinfunction "1")
 			(pintype "input")
+			(zone_connect 2)
 		)
 		(pad "1" thru_hole circle
@@
 			(pinfunction "1")
 			(pintype "input")
+			(zone_connect 2)
 		)
 		(pad "1" thru_hole circle
@@
 			(pinfunction "1")
 			(pintype "input")
+			(zone_connect 2)
 		)
 		(pad "1" thru_hole circle
@@
 			(pinfunction "1")
 			(pintype "input")
+			(zone_connect 2)
 		)
 	)
@@
 		(sheetname "Root")
 		(sheetfile "1280_modem.kicad_sch")
-		(attr smd)
+		(attr smd dnp)
 		(fp_line
 			(start -0.153641 -0.38)
@@
 			)
 		)
-		(property "Value" "10u"
+		(property "Value" "1u"
 			(at 0 1.43 90)
 			(layer "F.Fab")
@@
 			)
 		)
-		(property "Value" "AO3401A"
+		(property "Value" " DMP3056L-7 "
 			(at 0 2.4 90)
 			(layer "F.Fab")
@@
 		(sheetname "Root")
 		(sheetfile "1280_modem.kicad_sch")
-		(attr smd)
+		(attr smd dnp)
 		(fp_line
 			(start -0.107836 0.36)
@@
 			)
 		)
-		(property "Value" "100n"
+		(property "Value" "10n"
 			(at 0 1.43 0)
 			(layer "F.Fab")
@@
 			)
 		)
-		(property "Value" "10p"
+		(property "Value" "18p"
 			(at 0 1.43 90)
 			(layer "F.Fab")
@@
 			)
 		)
-		(property "Value" "13p"
+		(property "Value" "18p"
 			(at 0 1.43 90)
 			(layer "F.Fab")
@@
 			)
 		)
-		(property "Value" "470n"
+		(property "Value" "1u"
 			(at 0 1.43 0)
 			(layer "F.Fab")
@@
 			)
 		)
-		(property "Value" "10p"
+		(property "Value" "18p"
 			(at 0 1.43 90)
 			(layer "F.Fab")
@@
 			)
 		)
-		(property "Value" "10p"
+		(property "Value" "18p"
 			(at 0 1.43 90)
 			(layer "F.Fab")
@@
 			)
 		)
-		(property "mfn" "CX2016SA48000H0FLJG1"
+		(property "mfn" "FW520WFMT1"
 			(at 0 0 0)
 			(layer "F.Fab")
@@
 		(sheetname "Root")
 		(sheetfile "1280_modem.kicad_sch")
-		(attr smd)
+		(attr smd dnp)
 		(fp_line
 			(start -0.107836 0.36)
@@
 			)
 		)
-		(property "Value" "AO3401A"
+		(property "Value" " DMP3056L-7 "
 			(at 0 2.4 90)
 			(layer "F.Fab")
@@
 			)
 		)
-		(property "Value" "TCAN334"
+		(property "Value" "TCAN334GDCN"
 			(at 0 2.4 90)
 			(layer "F.Fab")
@@
 			)
 		)
-		(property ki_fp_filters "MountingHole*Pad*")
-		(sheetname "Root")
-		(sheetfile "1280_modem.kicad_sch")
 		(attr exclude_from_pos_files)
 		(fp_circle
@@
 			(pinfunction "1")
 			(pintype "input")
+			(zone_connect 2)
 		)
 		(pad "1" thru_hole circle
@@
 			(pinfunction "1")
 			(pintype "input")
+			(zone_connect 2)
 		)
 		(pad "1" thru_hole circle
@@
 			(pinfunction "1")
 			(pintype "input")
+			(zone_connect 2)
 		)
 		(pad "1" thru_hole circle
@@
 			(pinfunction "1")
 			(pintype "input")
+			(zone_connect 2)
 		)
 		(pad "1" thru_hole circle
@@
 			(pinfunction "1")
 			(pintype "input")
+			(zone_connect 2)
 		)
 		(pad "1" thru_hole circle
@@
 			(pinfunction "1")
 			(pintype "input")
+			(zone_connect 2)
 		)
 		(pad "1" thru_hole circle
@@
 			(pinfunction "1")
 			(pintype "input")
+			(zone_connect 2)
 		)
 		(pad "1" thru_hole circle
@@
 			(pinfunction "1")
 			(pintype "input")
+			(zone_connect 2)
 		)
 	)
@@
 			)
 		)
-		(property "Value" "13p"
+		(property "Value" "18p"
 			(at 0 1.43 0)
 			(layer "F.Fab")
@@
 			)
 		)
-		(property "Value" "14p"
+		(property "Value" "18p"
 			(at 0 -1.43 90)
 			(layer "B.Fab")
@@
 			)
 		)
-		(property "Value" "4u7"
+		(property "Value" "100n"
 			(at 0 -1.43 135)
 			(layer "B.Fab")
@@
 			)
 		)
-		(property ki_fp_filters "MountingHole*Pad*")
-		(sheetname "Root")
-		(sheetfile "1280_modem.kicad_sch")
 		(attr exclude_from_pos_files)
 		(fp_circle
@@
 			(pinfunction "1")
 			(pintype "input")
+			(zone_connect 2)
 		)
 		(pad "1" thru_hole circle
@@
 			(pinfunction "1")
 			(pintype "input")
+			(zone_connect 2)
 		)
 		(pad "1" thru_hole circle
@@
 			(pinfunction "1")
 			(pintype "input")
+			(zone_connect 2)
 		)
 		(pad "1" thru_hole circle
@@
 			(pinfunction "1")
 			(pintype "input")
+			(zone_connect 2)
 		)
 		(pad "1" thru_hole circle
@@
 			(pinfunction "1")
 			(pintype "input")
+			(zone_connect 2)
 		)
 		(pad "1" thru_hole circle
@@
 			(pinfunction "1")
 			(pintype "input")
+			(zone_connect 2)
 		)
 		(pad "1" thru_hole circle
@@
 			(pinfunction "1")
 			(pintype "input")
+			(zone_connect 2)
 		)
 		(pad "1" thru_hole circle
@@
 			(pinfunction "1")
 			(pintype "input")
+			(zone_connect 2)
 		)
 	)
@@
 			)
 		)
-		(property "Value" "4u7"
+		(property "Value" "100n"
 			(at 0 -1.43 135)
 			(layer "B.Fab")
@@
 			)
 		)
-		(property ki_fp_filters "MountingHole*Pad*")
-		(sheetname "Root")
-		(sheetfile "1280_modem.kicad_sch")
 		(attr exclude_from_pos_files)
 		(fp_circle
@@
 			(pinfunction "1")
 			(pintype "input")
+			(zone_connect 2)
 		)
 		(pad "1" thru_hole circle
@@
 			(pinfunction "1")
 			(pintype "input")
+			(zone_connect 2)
 		)
 		(pad "1" thru_hole circle
@@
 			(pinfunction "1")
 			(pintype "input")
+			(zone_connect 2)
 		)
 		(pad "1" thru_hole circle
@@
 			(pinfunction "1")
 			(pintype "input")
+			(zone_connect 2)
 		)
 		(pad "1" thru_hole circle
@@
 			(pinfunction "1")
 			(pintype "input")
+			(zone_connect 2)
 		)
 		(pad "1" thru_hole circle
@@
 			(pinfunction "1")
 			(pintype "input")
+			(zone_connect 2)
 		)
 		(pad "1" thru_hole circle
@@
 			(pinfunction "1")
 			(pintype "input")
+			(zone_connect 2)
 		)
 		(pad "1" thru_hole circle
@@
 			(pinfunction "1")
 			(pintype "input")
+			(zone_connect 2)
 		)
 	)
@@
 			)
 		)
-		(property "Value" "14p"
+		(property "Value" "18p"
 			(at 0 -1.43 0)
 			(layer "B.Fab")

Commit message: v1.1
Parts:
- removed the G*** at (99.6, 75.4)
- added R20: 330, Resistor_SMD:R_0603_1608Metric, B.Cu at (114.8, 63.0)
- added R21: 330, Resistor_SMD:R_0603_1608Metric, B.Cu at (116.6, 63.0)
- FL1: value RFBPF2012080AC2T00 -> DEA202450BT-1213C1
- Q1, Q2: value DMP3056L-7 -> DMP3056L-7
- moved R19 6.54 mm to (122.1, 63.3), turned to 90 degrees
Connections:
- D9 pad 1: Net-(D9-A) -> +3V3
- D9 pad 2: Earth -> Net-(D9-RK)
- D9 pad 3: /LED_G -> Net-(D9-GK)
- D9 pad 4: /LED_B -> Net-(D9-BK)
- R19 pad 1: Net-(D9-A) -> /LED_B
- R19 pad 2: +3V3 -> Net-(D9-BK)
- U1 pad 29: unconnected-(U1-PA8-Pad29) -> +3V3
- U1 pad 30: unconnected-(U1-PA9-Pad30) -> /2V8_EN
- U1 pad 31: unconnected-(U1-PA10-Pad31) -> Earth
- U2 pad 3: +3.3VA -> /2V8_EN
Routing:
- net /2V8_EN: track 0.00 -> 25.1 mm, vias 0 -> 2
- net +3V3: track 29.3 -> 43.2 mm, vias 7 -> 10
- net /LED_B: track 51.0 -> 39.1 mm
- net Net-(D9-BK): track 0.00 -> 9.91 mm
- net Net-(D9-GK): track 0.00 -> 7.23 mm
- net Net-(D9-RK): track 0.00 -> 2.92 mm
- net Net-(D9-A): track 2.69 -> 0.00 mm
- net Earth: track 220.8 -> 223.1 mm, vias 64 -> 65
- net /LED_G: track 41.5 -> 40.8 mm
- added copper zone on In2.Cu, net +3V3
Other:
- board text added: "V1.1 OCT 2025"
- board text removed: "V1.0 FEB 2024"
