File: hardware/1280_modem.kicad_sch (KiCad schematic)
At the start: 88 parts, among them IC1 SX1281IMLTRT, IC2 SKY65383-11, IC3 LMR50410Y3, J2 Conn_Coaxial, J2 jst gh 4, J5 jst gh 6, J8 USB_C_Receptacle_USB2.0, J9 jst_sh 6, Q1 AO3401A, Q2 AO3401A, U13 STM32U575CGTx, U2 TPS7A20285PDBVR, U2 USBLC6-2SC6, U4 TCAN334, Y1 48MHz, Y1 52MHz

Commit message: fix bom
Parts:
- C13, C14: value 14p -> 18p
- C21, C22: value 13p -> 18p
- U4: value TCAN334 -> TCAN334GDCN
- Y1: mfn CX2016SA48000H0FLJG1 -> FW520WFMT1
Changed lines of the file:
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@@
 			)
 		)
-		(property "Value" "14p"
+		(property "Value" "18p"
 			(at 100.33 96.52 0)
 			(effects
@@
 			)
 		)
-		(property "Value" "14p"
+		(property "Value" "18p"
 			(at 120.65 97.1613 0)
+			(do_not_autoplace yes)
 			(effects
 				(font
@@
 			)
 		)
-		(property "Value" "13p"
+		(property "Value" "18p"
 			(at 217.17 86.3663 0)
 			(effects
@@
 			)
 		)
-		(property "Value" "13p"
+		(property "Value" "18p"
 			(at 201.93 86.3663 0)
 			(effects
@@
 			)
 		)
-		(property "mfn" "CX2016SA48000H0FLJG1"
+		(property "mfn" "FW520WFMT1"
 			(at 209.55 78.74 0)
 			(effects
@@
 			)
 		)
-		(property "Value" "TCAN334"
+		(property "Value" "TCAN334GDCN"
 			(at 199.0441 162.56 0)
 			(effects

Commit message: final (?) bom
Parts:
- C11: value 4u7 -> 100n
- C15, C16, C17: value 10p -> 18p
- C27: value 10u -> 1u
- C32, C33, R4: now not fitted
- C6: value 100n -> 10n
- C7: value 470n -> 1u
- Q1, Q2: value AO3401A -> DMP3056L-7
Changed lines of the file:
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@@
 	(text "ok"
 		(exclude_from_sim no)
-		(at 195.58 46.99 0)
-		(effects
-			(font
-				(size 1.27 1.27)
-			)
-			(justify left bottom)
-		)
-	)
-	(text "ok"
-		(exclude_from_sim no)
 		(at 60.96 189.23 0)
 		(effects
@@
 		(fields_autoplaced yes)
 		(property "Reference" "C17"
-			(at 26.67 267.9763 0)
+			(at 26.67 267.9762 0)
 			(effects
 				(font
@@
 			)
 		)
-		(property "Value" "10p"
-			(at 26.67 270.5163 0)
+		(property "Value" "18p"
+			(at 26.67 270.5162 0)
 			(effects
 				(font
@@
 		(in_bom yes)
 		(on_board yes)
-		(dnp no)
+		(dnp yes)
 		(property "Reference" "C32"
 			(at 124.46 254.0063 0)
@@
 			)
 		)
-		(property "Value" "100n"
+		(property "Value" "10n"
 			(at 207.0163 57.15 90)
 			(effects
@@
 		(fields_autoplaced yes)
 		(property "Reference" "C27"
-			(at 175.26 218.4336 0)
+			(at 175.26 218.4335 0)
 			(effects
 				(font
@@
 			)
 		)
-		(property "Value" "10u"
-			(at 175.26 220.9736 0)
+		(property "Value" "1u"
+			(at 175.26 220.9735 0)
 			(effects
 				(font
@@
 		(fields_autoplaced yes)
 		(property "Reference" "C11"
-			(at 137.16 41.9163 0)
+			(at 137.16 41.9162 0)
 			(effects
 				(font
@@
 			)
 		)
-		(property "Value" "4u7"
-			(at 137.16 44.4563 0)
+		(property "Value" "100n"
+			(at 137.16 44.4562 0)
 			(effects
 				(font
@@
 		(fields_autoplaced yes)
 		(property "Reference" "C11"
-			(at 147.32 41.9163 0)
+			(at 147.32 41.9162 0)
 			(effects
 				(font
@@
 			)
 		)
-		(property "Value" "4u7"
-			(at 147.32 44.4563 0)
+		(property "Value" "100n"
+			(at 147.32 44.4562 0)
 			(effects
 				(font
@@
 		(fields_autoplaced yes)
 		(property "Reference" "C7"
-			(at 222.25 115.5763 0)
+			(at 222.25 115.5762 0)
 			(effects
 				(font
@@
 			)
 		)
-		(property "Value" "470n"
-			(at 222.25 118.1163 0)
+		(property "Value" "1u"
+			(at 222.25 118.1162 0)
 			(effects
 				(font
@@
 			)
 		)
-		(property "Value" "AO3401A"
+		(property "Value" " DMP3056L-7 "
 			(at 209.55 269.24 90)
 			(effects
@@
 		(in_bom yes)
 		(on_board yes)
-		(dnp no)
+		(dnp yes)
 		(property "Reference" "C33"
 			(at 115.57 237.4837 0)
@@
 		(fields_autoplaced yes)
 		(property "Reference" "C15"
-			(at 45.72 193.0463 0)
+			(at 45.72 193.0462 0)
 			(effects
 				(font
@@
 			)
 		)
-		(property "Value" "10p"
-			(at 45.72 195.5863 0)
+		(property "Value" "18p"
+			(at 45.72 195.5862 0)
 			(effects
 				(font
@@
 		(in_bom yes)
 		(on_board yes)
-		(dnp no)
+		(dnp yes)
 		(fields_autoplaced yes)
 		(property "Reference" "R4"
@@
 			)
 		)
-		(property "Value" "10p"
+		(property "Value" "18p"
 			(at 55.88 195.5863 0)
 			(effects
@@
 			)
 		)
-		(property "Value" "AO3401A"
+		(property "Value" " DMP3056L-7 "
 			(at 209.55 238.76 90)
 			(effects

Commit message: v1.1
Parts:
- added R20, R21: 330, Resistor_SMD:R_0603_1608Metric, symbol Device:R_Small
- FL1: value RFBPF2012080AC2T00 -> DEA202450BT-1213C1
- Q1, Q2: value DMP3056L-7 -> DMP3056L-7
- renumbered C12 to C1, C10 to C2, C11 to C25, C11 to C29, C13 to C3, C11 to C4, C14 to C5, J9 to J1, J8 to J3, J2 to J4, R27 to R1, R6 to R10, R18 to R2, R27 to R3, R13 to R9, U13 to U1, U2 to U3, Y1 to Y2
Connections:
- net +3.3VA: no longer U2.3 (EN)
- net +3V3: now also D9.1 (A), U1.29 (PA8); no longer R19.2
- net Earth: now also U1.31 (PA10), R21.1; no longer D9.2 (RK)
- net LED_B: now also R19.1; no longer D9.4 (BK)
- net LED_G: now also R20.1; no longer D9.3 (GK)
- net 2V8_EN: now reaches U1.30 (PA9)
- net 2V8_EN: now also U2.3 (EN)
- new net: D9.2 (RK), R21.2
- new net: D9.3 (GK), R20.2
- new net: D9.4 (BK), R19.2
- no-connect marks 10 -> 7
Other:
- moved on the sheet: D9
